Commit message: limo gazebo

File: limo_description/urdf/limo_four_diff.xacro (robot description, xacro)
@@ -37,4 +37,13 @@
         </collision>
     </link>
+    <!-- <link name="inertial_link">
+        <inertial>
+            <origin xyz="0.0 0.0 0.0" />
+            <mass value="${base_mass}" />
+            <inertia ixx="0" ixy="0" ixz="0"
+                     iyy="0" iyz="0"
+                     izz="0" />
+        </inertial>
+    </link> -->
     <link name="inertial_link">
         <inertial>
